File: Info-Robo-main-board.kicad_sch (KiCad schematic)
At the start: 20 parts, among them IC101 LM66100DCKT, IC102 LM66100DCKT, IC103 M78AR05-0.5, J101 XT60, J102 XH_4P, J103 XH_4P, J104 XH_4P, J105 XH_4P, J106 XH_4P, J107 XH_4P, J108 XH_4P, J109 XH_4P, U101 AMS1117-3.3

Commit message: complete design
Parts:
- removed J109: XH_4P, symbol Connector_Generic:Conn_01x04
- added D101, D102, D103, D104, D105: LED_Small, LED_SMD:LED_0402_1005Metric, symbol Device:LED_Small
- added D106, D107: POWER, LED_SMD:LED_0402_1005Metric, symbol Device:LED_Small
- added H101, H102, H103, H104: M3, MountingHole:MountingHole_3.2mm_M3, symbol Mechanical:MountingHole
- added J109, J110, J111, J112, J113, J114, J115, J116, J117, J118, J119, J120, J121, J122, J123, J124: XH_3P, Connector_JST:JST_XH_B3B-XH-A_1x03_P2.50mm_Vertical, symbol Connector_Generic:Conn_01x03
- added R101, R102, R103, R104, R105, R106, R107: 4.7k, Resistor_SMD:R_0402_1005Metric, symbol Device:R_Small
- C106: footprint Capacitor_THT:C_Disc_D3.8mm_W2.6mm_P2.50mm -> Capacitor_SMD:C_0402_1005Metric; LCSC (none) -> C307331
- C107: value 47uF -> 220uF; footprint Capacitor_THT:CP_Radial_D5.0mm_P2.50mm -> Capacitor_SMD:CP_Elec_10x10; LCSC (none) -> C125977
- J101: footprint Connector_AMASS:AMASS_XT60PW-M_1x02_P7.20mm_Horizontal -> Connector_AMASS:AMASS_XT60-M_1x02_P7.20mm_Vertical; LCSC (none) -> C19268037
- J102, J103, J104, J105, J106, J107, J108: footprint (none) -> Connector_JST:JST_XH_B4B-XH-A_1x04_P2.50mm_Vertical; LCSC (none) -> C595709
Connections:
- net +5V: now also J102.2 (Pin_2), J103.2 (Pin_2), J104.2 (Pin_2), J105.2 (Pin_2), J106.2 (Pin_2), J107.2 (Pin_2), J108.2 (Pin_2), J117.2 (Pin_2), J118.2 (Pin_2), J119.2 (Pin_2), J120.2 (Pin_2), J121.2 (Pin_2), J122.2 (Pin_2), J123.2 (Pin_2), J124.2 (Pin_2)
- net GND: now also J102.1 (Pin_1), J103.1 (Pin_1), J104.1 (Pin_1), J105.1 (Pin_1), J106.1 (Pin_1), J107.1 (Pin_1), J108.1 (Pin_1), J109.1 (Pin_1), J110.1 (Pin_1), J111.1 (Pin_1), J112.1 (Pin_1), J113.1 (Pin_1), J114.1 (Pin_1), J115.1 (Pin_1), J116.1 (Pin_1), J117.1 (Pin_1), J118.1 (Pin_1), J119.1 (Pin_1), J120.1 (Pin_1), J121.1 (Pin_1), J122.1 (Pin_1), J123.1 (Pin_1), J124.1 (Pin_1), R101.2, R102.2, R103.2, R104.2, R105.2, R106.2, R107.2
- net GPIO_in_PC0: now also J117.3 (Pin_3)
- net GPIO_in_PC1: now also J118.3 (Pin_3)
- net GPIO_in_PC13: now also J123.3 (Pin_3)
- net GPIO_in_PC15: now also J124.3 (Pin_3)
- net GPIO_in_PC2: now also J119.3 (Pin_3)
- net GPIO_in_PC3: now also J120.3 (Pin_3)
- net GPIO_in_PC4: now also J121.3 (Pin_3)
- net GPIO_in_PC5: now also J122.3 (Pin_3)
- net GPIO_out_PA15: now also D101.2 (A)
- net GPIO_out_PA4: now also J113.3 (Pin_3)
- net GPIO_out_PA8: now also J115.3 (Pin_3)
- net GPIO_out_PB14: now also J114.3 (Pin_3)
- net GPIO_out_PB4: now also D102.2 (A)
- net GPIO_out_PB5: now also D103.2 (A)
- net GPIO_out_PB6: now also D104.2 (A)
- net GPIO_out_PB7: now also D105.2 (A)
- net GPIO_out_PC6: now also J116.3 (Pin_3)
- net GPIO_out_PC7: now also J109.3 (Pin_3)
- net GPIO_out_PC8: now also J110.3 (Pin_3)
- net GPIO_out_PC9: now also J111.3 (Pin_3)
- net I2C_SCL: now also J106.3 (Pin_3)
- net I2C_SDA: now also J106.4 (Pin_4)
- net TIM2_CH1: now also J109.2 (Pin_2)
- net TIM2_CH3: now also J111.2 (Pin_2)
- net TIM2_CH4: now also J112.2 (Pin_2)
- net TIM3_CH1: now also J113.2 (Pin_2)
- net TIM3_CH2: now also J114.2 (Pin_2)
- net TIM3_CH3: now also J115.2 (Pin_2)
- net TIM3_CH4: now also J116.2 (Pin_2)
- net UART3_RX: now also J104.4 (Pin_4)
- net UART3_TX: now also J104.3 (Pin_3)
- net UART4_RX: now also J102.4 (Pin_4)
- net UART4_TX: now also J102.3 (Pin_3)
- net UART5_RX: now also J105.4 (Pin_4)
- net UART5_TX: now also J105.3 (Pin_3)
- net USART1_RX: now also J103.4 (Pin_4)
- net USART1_TX: now also J103.3 (Pin_3)
- net VBUS_USB: now also D106.2 (A)
- net VIN: now also D107.2 (A)
- net CAN2/CANH: now reaches J108.3 (Pin_3)
- net CAN2/CANL: now reaches J108.4 (Pin_4)
- net CAN1/CANH: now reaches J107.3 (Pin_3)
- net CAN1/CANL: now reaches J107.4 (Pin_4)
- new net: D101.1 (K), R101.1
- new net: D105.1 (K), R105.1
- new net: D102.1 (K), R102.1
- new net: D103.1 (K), R103.1
- new net: D106.1 (K), R106.1
- new net: D104.1 (K), R104.1
- new net: D107.1 (K), R107.1
- new net GPIO_out_PB15: J112.3 (Pin_3)
- new net TIM2_CH2: J110.2 (Pin_2)
Other:
- added sheet CAN1 (MCP2562.kicad_sch)
- added sheet CAN2 (MCP2562.kicad_sch)
- moved on the sheet: J102, J103, J104, J105, J106, J107, J108
